File: ADSR.sch (KiCad schematic (older format))
At the start: 46 parts, among them P15 1M, P16 10k, P17 R_POT, P18 1M, U11 UA747, U7 UA747

Commit message: Annotate
Parts:
- gave numbers to parts that had none: 39
Changed lines of the file:
@@
 $EndComp
 $Comp
-L Device:R R?
+L Device:R R4
 U 1 1 5E33E8C9
 P 3900 3100
-F 0 "R?" H 3970 3146 50  0000 L CNN
+F 0 "R4" H 3970 3146 50  0000 L CNN
 F 1 "33k" H 3970 3055 50  0000 L CNN
 F 2 "" V 3830 3100 50  0001 C CNN
@@
 	3900 2950 4100 2950
 $Comp
-L Device:R R?
+L Device:R R3
 U 1 1 5E33EF6B
 P 3600 3100
-F 0 "R?" H 3670 3146 50  0000 L CNN
+F 0 "R3" H 3670 3146 50  0000 L CNN
 F 1 "91k" H 3670 3055 50  0000 L CNN
 F 2 "" V 3530 3100 50  0001 C CNN
@@
 $EndComp
 $Comp
-L Device:R R?
+L Device:R R9
 U 1 1 5E33FFB4
 P 6400 900
-F 0 "R?" H 6470 946 50  0000 L CNN
+F 0 "R9" H 6470 946 50  0000 L CNN
 F 1 "9k1" H 6470 855 50  0000 L CNN
 F 2 "" V 6330 900 50  0001 C CNN
@@
 	7550 1850 7350 1850
 $Comp
-L Device:Q_NPN_BCE Q?
+L Device:Q_NPN_BCE Q1
 U 1 1 5E34CF9A
 P 6850 3050
-F 0 "Q?" H 7041 3096 50  0000 L CNN
+F 0 "Q1" H 7041 3096 50  0000 L CNN
 F 1 "BC184" H 7041 3005 50  0000 L CNN
 F 2 "" H 7050 3150 50  0001 C CNN
@@
 Connection ~ 3900 2950
 $Comp
-L Device:R R?
+L Device:R R5
 U 1 1 5E34E905
 P 4350 2250
-F 0 "R?" V 4143 2250 50  0000 C CNN
+F 0 "R5" V 4143 2250 50  0000 C CNN
 F 1 "10k" V 4234 2250 50  0000 C CNN
 F 2 "" V 4280 2250 50  0001 C CNN
@@
 	6200 3300 6200 2850
 $Comp
-L Device:R R?
+L Device:R R6
 U 1 1 5E354935
 P 6050 3600
-F 0 "R?" H 6120 3646 50  0000 L CNN
+F 0 "R6" H 6120 3646 50  0000 L CNN
 F 1 "1k5" H 6120 3555 50  0000 L CNN
 F 2 "" V 5980 3600 50  0001 C CNN
@@
 $EndComp
 $Comp
-L Device:D D?
+L Device:D D3
 U 1 1 5E355032
 P 6050 3900
-F 0 "D?" V 6004 3979 50  0000 L CNN
+F 0 "D3" V 6004 3979 50  0000 L CNN
 F 1 "1N4148" V 6095 3979 50  0000 L CNN
 F 2 "" H 6050 3900 50  0001 C CNN
@@
 $EndComp
 $Comp
-L Device:CP C?
+L Device:CP C1
 U 1 1 5E355590
 P 6450 4800
-F 0 "C?" H 6568 4846 50  0000 L CNN
+F 0 "C1" H 6568 4846 50  0000 L CNN
 F 1 "10uF" H 6568 4755 50  0000 L CNN
 F 2 "" H 6488 4650 50  0001 C CNN
@@
 $EndComp
 $Comp
-L Device:R R?
+L Device:R R11
 U 1 1 5E356794
 P 6750 3850
-F 0 "R?" H 6820 3896 50  0000 L CNN
+F 0 "R11" H 6820 3896 50  0000 L CNN
 F 1 "330" H 6820 3805 50  0000 L CNN
 F 2 "" V 6680 3850 50  0001 C CNN
@@
 $EndComp
 $Comp
-L Device:D D?
+L Device:D D4
 U 1 1 5E35679A
 P 6750 4150
-F 0 "D?" V 6704 4229 50  0000 L CNN
+F 0 "D4" V 6704 4229 50  0000 L CNN
 F 1 "1N4148" V 6795 4229 50  0000 L CNN
 F 2 "" H 6750 4150 50  0001 C CNN
@@
 Connection ~ 6050 2850
 $Comp
-L Device:Q_NPN_BCE Q?
+L Device:Q_NPN_BCE Q5
 U 1 1 5E35BE62
 P 8550 1400
-F 0 "Q?" H 8741 1446 50  0000 L CNN
+F 0 "Q5" H 8741 1446 50  0000 L CNN
 F 1 "BC184" H 8741 1355 50  0000 L CNN
 F 2 "" H 8750 1500 50  0001 C CNN
@@
 $EndComp
 $Comp
-L Device:Q_NPN_BCE Q?
+L Device:Q_NPN_BCE Q2
 U 1 1 5E35C151
 P 7750 4600
-F 0 "Q?" H 7941 4646 50  0000 L CNN
+F 0 "Q2" H 7941 4646 50  0000 L CNN
 F 1 "BC184" H 7941 4555 50  0000 L CNN
 F 2 "" H 7950 4700 50  0001 C CNN
@@
 $EndComp
 $Comp
-L Device:Q_NPN_BCE Q?
+L Device:Q_NPN_BCE Q6
 U 1 1 5E35C593
 P 9850 1400
-F 0 "Q?" H 10041 1446 50  0000 L CNN
+F 0 "Q6" H 10041 1446 50  0000 L CNN
 F 1 "BC184" H 10041 1355 50  0000 L CNN
 F 2 "" H 10050 1500 50  0001 C CNN
@@
 $EndComp
 $Comp
-L Device:R R?
+L Device:R R20
 U 1 1 5E35CBA0
 P 8450 950
-F 0 "R?" H 8520 996 50  0000 L CNN
+F 0 "R20" H 8520 996 50  0000 L CNN
 F 1 "5k1" H 8520 905 50  0000 L CNN
 F 2 "" V 8380 950 50  0001 C CNN
@@
 $EndComp
 $Comp
-L Device:R R?
+L Device:R R1
 U 1 1 5E35E2F2
 P 2850 1700
-F 0 "R?" H 2920 1746 50  0000 L CNN
+F 0 "R1" H 2920 1746 50  0000 L CNN
 F 1 "10k" H 2920 1655 50  0000 L CNN
 F 2 "" V 2780 1700 50  0001 C CNN
@@
 $EndComp
 $Comp
-L Device:R R?
+L Device:R R2
 U 1 1 5E35DDB3
 P 2850 2100
-F 0 "R?" H 2920 2146 50  0000 L CNN
+F 0 "R2" H 2920 2146 50  0000 L CNN
 F 1 "5k1" H 2920 2055 50  0000 L CNN
 F 2 "" V 2780 2100 50  0001 C CNN
@@
 $EndComp
 $Comp
-L Switch:SW_SPDT SW?
+L Switch:SW_SPDT SW1
 U 1 1 5E3617B9
 P 3400 2750
-F 0 "SW?" H 3400 2425 50  0000 C CNN
+F 0 "SW1" H 3400 2425 50  0000 C CNN
 F 1 "SW_SPDT" H 3400 2516 50  0000 C CNN
 F 2 "" H 3400 2750 50  0001 C CNN
@@
 	8450 1100 8450 1150
 $Comp
-L Device:R R?
+L Device:R R23
 U 1 1 5E36742E
 P 9100 950
-F 0 "R?" H 9170 996 50  0000 L CNN
+F 0 "R23" H 9170 996 50  0000 L CNN
 F 1 "91k" H 9170 905 50  0000 L CNN
 F 2 "" V 9030 950 50  0001 C CNN
@@
 	9100 1100 9100 1150
 $Comp
-L Device:C C?
+L Device:C C2
 U 1 1 5E3680BB
 P 8800 1150
-F 0 "C?" V 8548 1150 50  0000 C CNN
+F 0 "C2" V 8548 1150 50  0000 C CNN
 F 1 "10nF" V 8639 1150 50  0000 C CNN
 F 2 "" H 8838 1000 50  0001 C CNN
@@
 	8450 1150 8450 1200
 $Comp
-L Device:R R?
+L Device:R R24
 U 1 1 5E36AAB6
 P 9650 1150
-F 0 "R?" V 9443 1150 50  0000 C CNN
+F 0 "R24" V 9443 1150 50  0000 C CNN
 F 1 "91k" V 9534 1150 50  0000 C CNN
 F 2 "" V 9580 1150 50  0001 C CNN
@@
 	9950 1150 9950 1200
 $Comp
-L Device:R R?
+L Device:R R26
 U 1 1 5E36E31B
 P 9950 950
-F 0 "R?" H 10020 996 50  0000 L CNN
+F 0 "R26" H 10020 996 50  0000 L CNN
 F 1 "5k1" H 10020 905 50  0000 L CNN
 F 2 "" V 9880 950 50  0001 C CNN
@@
 $EndComp
 $Comp
-L Device:R R?
+L Device:R R14
 U 1 1 5E3729D6
 P 7300 3050
-F 0 "R?" V 7093 3050 50  0000 C CNN
+F 0 "R14" V 7093 3050 50  0000 C CNN
 F 1 "27k" V 7184 3050 50  0000 C CNN
 F 2 "" V 7230 3050 50  0001 C CNN
@@
 $EndComp
 $Comp
-L Device:R R?
+L Device:R R16
 U 1 1 5E375A78
 P 8050 3050
-F 0 "R?" V 7843 3050 50  0000 C CNN
+F 0 "R16" V 7843 3050 50  0000 C CNN
 F 1 "100k" V 7934 3050 50  0000 C CNN
 F 2 "" V 7980 3050 50  0001 C CNN
@@
 $EndComp
 $Comp
-L Device:Q_NPN_BCE Q?
+L Device:Q_NPN_BCE Q4
 U 1 1 5E377C04
 P 8500 3050
-F 0 "Q?" H 8691 3096 50  0000 L CNN
+F 0 "Q4" H 8691 3096 50  0000 L CNN
 F 1 "BC184" H 8691 3005 50  0000 L CNN
 F 2 "" H 8700 3150 50  0001 C CNN
@@
 	7650 3050 7900 3050
 $Comp
-L Device:R R?
+L Device:R R19
 U 1 1 5E3A496C
 P 8100 4950
-F 0 "R?" H 8170 4996 50  0000 L CNN
+F 0 "R19" H 8170 4996 50  0000 L CNN
 F 1 "33k" H 8170 4905 50  0000 L CNN
 F 2 "" V 8030 4950 50  0001 C CNN
@@
 	8100 4600 7950 4600
 $Comp
-L Device:D D?
+L Device:D D5
 U 1 1 5E3A9482
 P 8100 5400
-F 0 "D?" V 8054 5479 50  0000 L CNN
+F 0 "D5" V 8054 5479 50  0000 L CNN
 F 1 "D" V 8145 5479 50  0000 L CNN
 F 2 "" H 8100 5400 50  0001 C CNN
@@
 	8100 5250 8100 5100
 $Comp
-L Device:R R?
+L Device:R R18
 U 1 1 5E3AB131
 P 8100 4350
-F 0 "R?" H 8170 4396 50  0000 L CNN
+F 0 "R18" H 8170 4396 50  0000 L CNN
 F 1 "100k" H 8170 4305 50  0000 L CNN
 F 2 "" V 8030 4350 50  0001 C CNN
@@
 $EndComp
 $Comp
-L Device:R R?
+L Device:R R17
 U 1 1 5E3AB83B
 P 8100 3950
-F 0 "R?" H 8170 3996 50  0000 L CNN
+F 0 "R17" H 8170 3996 50  0000 L CNN
 F 1 "68k" H 8170 3905 50  0000 L CNN
 F 2 "" V 8030 3950 50  0001 C CNN
@@
 Connection ~ 9100 1150
 $Comp
-L Device:R R?
+L Device:R R21
 U 1 1 5E3B1A18
 P 8600 2550
-F 0 "R?" H 8670 2596 50  0000 L CNN
+F 0 "R21" H 8670 2596 50  0000 L CNN
 F 1 "27k" H 8670 2505 50  0000 L CNN
 F 2 "" V 8530 2550 50  0001 C CNN
@@
 	8100 4150 8100 4200
 $Comp
-L Device:Q_NPN_BCE Q?
+L Device:Q_NPN_BCE Q3
 U 1 1 5E3BA7D2
 P 8000 2050
-F 0 "Q?" H 8191 2004 50  0000 L CNN
+F 0 "Q3" H 8191 2004 50  0000 L CNN
 F 1 "BC184" H 8191 2095 50  0000 L CNN
 F 2 "" H 8200 2150 50  0001 C CNN
@@
 Connection ~ 5700 5900
 $Comp
-L Device:R R?
+L Device:R R13
 U 1 1 5E3D3470
 P 6800 6300
-F 0 "R?" H 6870 6346 50  0000 L CNN
+F 0 "R13" H 6870 6346 50  0000 L CNN
 F 1 "5k1" H 6870 6255 50  0000 L CNN
 F 2 "" V 6730 6300 50  0001 C CNN
@@
 $EndComp
 $Comp
-L Device:R R?
+L Device:R R12
 U 1 1 5E3D3DD4
 P 6800 5500
-F 0 "R?" H 6870 5546 50  0000 L CNN
+F 0 "R12" H 6870 5546 50  0000 L CNN
 F 1 "10k" H 6870 5455 50  0000 L CNN
 F 2 "" V 6730 5500 50  0001 C CNN
@@
 Connection ~ 6050 4650
 $Comp
-L Device:D D?
+L Device:D D1
 U 1 1 5E6C2F34
 P 5900 4800
-F 0 "D?" V 5854 4879 50  0000 L CNN
+F 0 "D1" V 5854 4879 50  0000 L CNN
 F 1 "D" V 5945 4879 50  0000 L CNN
 F 2 "" H 5900 4800 50  0001 C CNN
@@
 $EndComp
 $Comp
-L Device:R R?
+L Device:R R15
 U 1 1 5E6C4FCC
 P 7650 2800
-F 0 "R?" H 7720 2846 50  0000 L CNN
+F 0 "R15" H 7720 2846 50  0000 L CNN
 F 1 "6k8" H 7720 2755 50  0000 L CNN
 F 2 "" V 7580 2800 50  0001 C CNN
@@
 	7650 2550 7650 2650
 $Comp
-L Device:R R?
+L Device:R R25
 U 1 1 5E6D2566
 P 9800 2300
-F 0 "R?" V 9593 2300 50  0000 C CNN
+F 0 "R25" V 9593 2300 50  0000 C CNN
 F 1 "27k" V 9684 2300 50  0000 C CNN
 F 2 "" V 9730 2300 50  0001 C CNN
@@
 	8900 1400 9000 1400
 $Comp
-L Device:R R?
+L Device:R R22
 U 1 1 5E6E124F
 P 8700 1900
-F 0 "R?" V 8493 1900 50  0000 C CNN
+F 0 "R22" V 8493 1900 50  0000 C CNN
 F 1 "27k" V 8584 1900 50  0000 C CNN
 F 2 "" V 8630 1900 50  0001 C CNN
@@
 ENVELOPE_OUT
 $Comp
-L Device:R R?
+L Device:R R7
 U 1 1 5E6EDB1A
 P 6150 6300
-F 0 "R?" H 6220 6346 50  0000 L CNN
+F 0 "R7" H 6220 6346 50  0000 L CNN
 F 1 "470" H 6220 6255 50  0000 L CNN
 F 2 "" V 6080 6300 50  0001 C CNN
@@
 	6650 2550 7100 2550
 $Comp
-L Device:R R?
+L Device:R R8
 U 1 1 5E71967D
 P 6350 2400
-F 0 "R?" H 6420 2446 50  0000 L CNN
+F 0 "R8" H 6420 2446 50  0000 L CNN
 F 1 "1k5" H 6420 2355 50  0000 L CNN
 F 2 "" V 6280 2400 50  0001 C CNN
@@
 $EndComp
 $Comp
-L Device:D D?
+L Device:D D2
 U 1 1 5E719683
 P 6050 2400
-F 0 "D?" V 6004 2479 50  0000 L CNN
+F 0 "D2" V 6004 2479 50  0000 L CNN
 F 1 "1N4148" V 6095 2479 50  0000 L CNN
 F 2 "" H 6050 2400 50  0001 C CNN

Commit message: VCF work
Connections:
- net labels added: ENVELOPE
- net labels removed: ENVELOPE_OUT
Changed lines of the file:
@@
 	8850 1900 8900 1900
 Text GLabel 5900 6700 0    50   Output ~ 0
-ENVELOPE_OUT
+ENVELOPE
 $Comp
 L Device:R R7

Commit message: VCF work
Parts:
- U11, U7: symbol Amplifier_Operational:UA747 -> janel-panel-minimoog-rescue:UA747-Amplifier_Operational
Changed lines of the file:
@@
 $EndDescr
 $Comp
-L Amplifier_Operational:UA747 U7
+L janel-panel-minimoog-rescue:UA747-Amplifier_Operational U7
 U 1 1 5E33ACAE
 P 4400 2850
+AR Path="/5E33ACAE" Ref="U7"  Part="1"
+AR Path="/5E33A92B/5E33ACAE" Ref="U7"  Part="1"
 F 0 "U7" H 4744 2896 50  0000 L CNN
 F 1 "UA747" H 4744 2805 50  0000 L CNN
@@
 $EndComp
 $Comp
-L Amplifier_Operational:UA747 U7
+L janel-panel-minimoog-rescue:UA747-Amplifier_Operational U7
 U 2 1 5E33BB06
 P 7050 1850
+AR Path="/5E33BB06" Ref="U7"  Part="2"
+AR Path="/5E33A92B/5E33BB06" Ref="U7"  Part="2"
 F 0 "U7" H 7394 1896 50  0000 L CNN
 F 1 "UA747" H 7394 1805 50  0000 L CNN
@@
 	8600 2050 8600 2400
 $Comp
-L Amplifier_Operational:UA747 U11
+L janel-panel-minimoog-rescue:UA747-Amplifier_Operational U11
 U 1 1 5E3BE335
 P 5000 5900
+AR Path="/5E3BE335" Ref="U11"  Part="1"
+AR Path="/5E33A92B/5E3BE335" Ref="U11"  Part="1"
 F 0 "U11" H 5344 5946 50  0000 L CNN
 F 1 "UA747" H 5344 5855 50  0000 L CNN
@@
 	4900 6300 4900 6200
 $Comp
-L Amplifier_Operational:UA747 U11
+L janel-panel-minimoog-rescue:UA747-Amplifier_Operational U11
 U 2 1 5E3BF552
 P 7250 5900
+AR Path="/5E3BF552" Ref="U11"  Part="2"
+AR Path="/5E33A92B/5E3BF552" Ref="U11"  Part="2"
 F 0 "U11" H 7594 5946 50  0000 L CNN
 F 1 "UA747" H 7594 5855 50  0000 L CNN

Commit message: Update some components
Parts:
- renumbered C1 to C12, C2 to C13, D1 to D3, D2 to D4, D3 to D5, D4 to D6, D5 to D7, P15 to P5, P16 to P6, P18 to P7, P17 to P8, Q2 to Q10, Q3 to Q11, Q4 to Q12, Q5 to Q13, Q6 to Q14, Q1 to Q9, R1 to R47, R2 to R48, R3 to R49, R4 to R50, R5 to R51, R6 to R52, R7 to R53, R8 to R54, R9 to R55, R10 to R56, R11 to R57, R12 to R58, R13 to R59, R14 to R60, R15 to R61, R16 to R62, R17 to R63, R18 to R64, R19 to R65, R20 to R66, R21 to R67, R22 to R68, R23 to R69, R24 to R70, R25 to R71, R26 to R72, U7 to U6, U11 to U7
Connections:
- no-connect marks 6 -> 0

Commit message: Create pcb and other updates
Parts:
- C12: footprint (none) -> Capacitor_THT:CP_Radial_D6.3mm_P2.50mm
- C13: footprint (none) -> Capacitor_THT:C_Disc_D5.0mm_W2.5mm_P5.00mm
- D3, D4, D5, D6, D7: footprint (none) -> Diode_THT:D_DO-15_P12.70mm_Horizontal
- K5: renamed from SW1; footprint (none) -> Connector_PinSocket_2.54mm:PinSocket_1x03_P2.54mm_Vertical
- P15: renamed from P5; footprint (none) -> Connector_PinSocket_2.54mm:PinSocket_1x03_P2.54mm_Vertical
- P17: renamed from P8; footprint (none) -> Connector_PinSocket_2.54mm:PinSocket_1x03_P2.54mm_Vertical
- P18: renamed from P7; footprint (none) -> Connector_PinSocket_2.54mm:PinSocket_1x03_P2.54mm_Vertical
- P6: footprint (none) -> Connector_PinSocket_2.54mm:PinSocket_1x03_P2.54mm_Vertical
- Q10, Q11, Q12, Q13, Q14, Q9: footprint (none) -> Package_TO_SOT_THT:TO-92L_Inline_Wide
- R47, R48, R49, R50, R51, R52, R53, R54, R55, R57, R58, R59, R60, R61, R62, R63, R64, R65, R66, R67, R68, R69, R70, R71, R72: footprint (none) -> Resistor_THT:R_Axial_DIN0207_L6.3mm_D2.5mm_P10.16mm_Horizontal
- RV56: renamed from R56; footprint (none) -> Potentiometer_THT:Potentiometer_Bourns_3296W_Vertical
- U11: renamed from U7; footprint (none) -> Package_DIP:DIP-14_W7.62mm_Socket_LongPads
- U7: renamed from U6; footprint (none) -> Package_DIP:DIP-14_W7.62mm_Socket_LongPads
Other:
- moved on the sheet: U11A
