File: Keyboard.sch (KiCad schematic (older format))
At the start: 31 parts, among them K6 SW_SPST, P7 1M

Commit message: Annotate
Parts:
- gave numbers to parts that had none: 28

Commit message: VCF work
Parts:
- U1: symbol Amplifier_Operational:uA741-DIP14 -> janel-panel-minimoog-rescue:uA741-DIP14-Amplifier_Operational
Changed lines of the file:
@@
 $EndComp
 $Comp
-L Amplifier_Operational:uA741-DIP14 U1
+L janel-panel-minimoog-rescue:uA741-DIP14-Amplifier_Operational U1
 U 1 1 5E382580
 P 3850 2600

Commit message: Update some components
Parts:
- renumbered C1 to C14, C2 to C15, C3 to C16, C4 to C17, D1 to D8, D2 to D9, K6 to K5, P7 to P9, Q1 to Q15, Q2 to Q16, Q3 to Q17, Q4 to Q18, Q5 to Q19, R1 to R73, R6 to R74, R2 to R75, R3 to R76, R4 to R77, R5 to R78, R7 to R79, R8 to R80, R9 to R81, R10 to R82, R11 to R83, R12 to R84, R13 to R85, R14 to R86, R15 to R87, R16 to R88, R17 to R89, U1 to U8

Commit message: ERC pass
Parts:
- added J1: Conn_01x05_Male, symbol Connector:Conn_01x05_Male
Connections:
- net +5V: now also J1.4 (Pin_4)
- net A: now also J1.2 (Pin_2); no longer R77.1
- net B: now also J1.5 (Pin_5)
- net C: now also J1.3 (Pin_3)
- new net D: J1.1 (Pin_1), R77.1
Other:
- moved on the sheet: R77
Changed lines of the file:
@@
 Wire Wire Line
 	1250 1250 1250 1300
-Text GLabel 1000 2400 0    50   Input ~ 0
+Text GLabel 1250 1800 0    50   Input ~ 0
 A
-Wire Wire Line
-	1000 2400 1100 2400
-Wire Wire Line
-	1100 2400 1100 1800
-Wire Wire Line
-	1100 1800 1250 1800
 Wire Wire Line
 	1250 1800 1250 1700
@@
 L power:GND #PWR054
 U 1 1 5E3AE014
-P 1250 2250
-F 0 "#PWR054" H 1250 2000 50  0001 C CNN
-F 1 "GND" H 1255 2077 50  0000 C CNN
-F 2 "" H 1250 2250 50  0001 C CNN
-F 3 "" H 1250 2250 50  0001 C CNN
-	1    1250 2250
+P 1600 2400
+F 0 "#PWR054" H 1600 2150 50  0001 C CNN
+F 1 "GND" H 1605 2227 50  0000 C CNN
+F 2 "" H 1600 2400 50  0001 C CNN
+F 3 "" H 1600 2400 50  0001 C CNN
+	1    1600 2400
 	1    0    0    -1
 $EndComp
@@
 L Device:R R77
 U 1 1 5E3AE68C
-P 1250 2050
-F 0 "R77" H 1320 2096 50  0000 L CNN
-F 1 "31.6" H 1320 2005 50  0000 L CNN
-F 2 "" V 1180 2050 50  0001 C CNN
-F 3 "~" H 1250 2050 50  0001 C CNN
-	1    1250 2050
-	1    0    0    -1
-$EndComp
-Wire Wire Line
-	1250 1900 1250 1850
-Connection ~ 1250 1800
-Wire Wire Line
-	1250 2200 1250 2250
-Text GLabel 1600 2400 2    50   Input ~ 0
+P 1600 2200
+F 0 "R77" H 1670 2246 50  0000 L CNN
+F 1 "31.6" H 1670 2155 50  0000 L CNN
+F 2 "" V 1530 2200 50  0001 C CNN
+F 3 "~" H 1600 2200 50  0001 C CNN
+	1    1600 2200
+	1    0    0    -1
+$EndComp
+Wire Wire Line
+	1600 2050 1600 2000
+Wire Wire Line
+	1600 2350 1600 2400
+Text GLabel 1600 2000 2    50   Input ~ 0
 D
-Wire Wire Line
-	1600 2400 1600 1850
-Wire Wire Line
-	1600 1850 1250 1850
-Connection ~ 1250 1850
-Wire Wire Line
-	1250 1850 1250 1800
 Text GLabel 2650 2050 0    50   Input ~ 0
 B
@@
 	1    0    0    -1
 $EndComp
+Text GLabel 1150 3000 2    50   Input ~ 0
+A
+Text GLabel 1150 3300 2    50   Input ~ 0
+B
+Text GLabel 1150 3100 2    50   Input ~ 0
+C
+$Comp
+L power:+5V #PWR0129
+U 1 1 5E9D6C88
+P 1150 3200
+F 0 "#PWR0129" H 1150 3050 50  0001 C CNN
+F 1 "+5V" H 1165 3373 50  0000 C CNN
+F 2 "" H 1150 3200 50  0001 C CNN
+F 3 "" H 1150 3200 50  0001 C CNN
+	1    1150 3200
+	0    1    1    0
+$EndComp
+$Comp
+L Connector:Conn_01x05_Male J1
+U 1 1 5E9DA8F7
+P 950 3100
+F 0 "J1" H 1058 3481 50  0000 C CNN
+F 1 "Conn_01x05_Male" H 1058 3390 50  0000 C CNN
+F 2 "" H 950 3100 50  0001 C CNN
+F 3 "~" H 950 3100 50  0001 C CNN
+	1    950  3100
+	1    0    0    -1
+$EndComp
+Text GLabel 1150 2900 2    50   Input ~ 0
+D
 $EndSCHEMATC

Commit message: Create pcb and other updates
Parts:
- C14, C15: footprint (none) -> Capacitor_THT:C_Disc_D5.0mm_W2.5mm_P5.00mm
- C16, C17: footprint (none) -> Capacitor_THT:CP_Radial_D6.3mm_P2.50mm
- D8, D9: footprint (none) -> Diode_THT:D_DO-15_P12.70mm_Horizontal
- J1: footprint (none) -> Connector_PinHeader_2.54mm:PinHeader_1x05_P2.54mm_Vertical
- K6: renamed from K5; footprint (none) -> Connector_PinSocket_2.54mm:PinSocket_1x03_P2.54mm_Vertical
- P7: renamed from P9; footprint (none) -> Connector_PinSocket_2.54mm:PinSocket_1x03_P2.54mm_Vertical; Label (none) -> GLIDE
- Q15: footprint (none) -> Package_TO_SOT_THT:TO-92L_Inline_Wide
- Q16, Q17, Q18, Q19: footprint Package_TO_SOT_THT:TO-92_Inline -> Package_TO_SOT_THT:TO-92L_Inline_Wide
- R73, R75, R76, R77, R78, R79, R80, R81, R82, R83, R84, R85, R86, R87, R88, R89: footprint (none) -> Resistor_THT:R_Axial_DIN0207_L6.3mm_D2.5mm_P10.16mm_Horizontal
- RV74: renamed from R74; footprint (none) -> Potentiometer_THT:Potentiometer_Bourns_3296W_Vertical
- U3: renamed from U8; footprint (none) -> Package_DIP:DIP-14_W7.62mm_Socket_LongPads
Changed lines of the file:
@@
 F 0 "R73" H 870 1146 50  0000 L CNN
 F 1 "150" H 870 1055 50  0000 L CNN
-F 2 "" V 730 1100 50  0001 C CNN
+F 2 "Resistor_THT:R_Axial_DIN0207_L6.3mm_D2.5mm_P10.16mm_Horizontal" V 730 1100 50  0001 C CNN
 F 3 "~" H 800 1100 50  0001 C CNN
 	1    800  1100
@@
 F 0 "R75" H 870 1896 50  0000 L CNN
 F 1 "9k1" H 870 1805 50  0000 L CNN
-F 2 "" V 730 1850 50  0001 C CNN
+F 2 "Resistor_THT:R_Axial_DIN0207_L6.3mm_D2.5mm_P10.16mm_Horizontal" V 730 1850 50  0001 C CNN
 F 3 "~" H 800 1850 50  0001 C CNN
 	1    800  1850
@@
 $EndComp
 $Comp
-L Device:R_POT_TRIM R74
+L Device:R_POT_TRIM RV74
 U 1 1 5E37BB25
 P 800 1500
-F 0 "R74" H 731 1546 50  0000 R CNN
+F 0 "RV74" H 731 1546 50  0000 R CNN
 F 1 "330" H 731 1455 50  0000 R CNN
-F 2 "" H 800 1500 50  0001 C CNN
+F 2 "Potentiometer_THT:Potentiometer_Bourns_3296W_Vertical" H 800 1500 50  0001 C CNN
 F 3 "~" H 800 1500 50  0001 C CNN
 	1    800  1500
@@
 F 0 "Q15" H 1340 1454 50  0000 L CNN
 F 1 "Q_PNP_BCE" H 1340 1545 50  0000 L CNN
-F 2 "" H 1350 1600 50  0001 C CNN
+F 2 "Package_TO_SOT_THT:TO-92L_Inline_Wide" H 1350 1600 50  0001 C CNN
 F 3 "~" H 1150 1500 50  0001 C CNN
 	1    1150 1500
@@
 F 0 "R76" H 1320 1146 50  0000 L CNN
 F 1 "220" H 1320 1055 50  0000 L CNN
-F 2 "" V 1180 1100 50  0001 C CNN
+F 2 "Resistor_THT:R_Axial_DIN0207_L6.3mm_D2.5mm_P10.16mm_Horizontal" V 1180 1100 50  0001 C CNN
 F 3 "~" H 1250 1100 50  0001 C CNN
 	1    1250 1100
@@
 F 0 "C16" H 10318 1196 50  0000 L CNN
 F 1 "1uF" H 10318 1105 50  0000 L CNN
-F 2 "" H 10238 1000 50  0001 C CNN
+F 2 "Capacitor_THT:CP_Radial_D6.3mm_P2.50mm" H 10238 1000 50  0001 C CNN
 F 3 "~" H 10200 1150 50  0001 C CNN
 	1    10200 1150
@@
 $EndComp
 $Comp
-L Switch:SW_SPST K5
+L Switch:SW_SPST K6
 U 1 1 5E37FB91
 P 2800 1850
-F 0 "K5" V 2754 1948 50  0000 L CNN
+F 0 "K6" V 2754 1948 50  0000 L CNN
 F 1 "SW_SPST" V 2845 1948 50  0000 L CNN
-F 2 "" H 2800 1850 50  0001 C CNN
+F 2 "Connector_PinSocket_2.54mm:PinSocket_1x03_P2.54mm_Vertical" H 2800 1850 50  0001 C CNN
 F 3 "~" H 2800 1850 50  0001 C CNN
 	1    2800 1850
@@
 F 0 "R78" H 2870 2346 50  0000 L CNN
 F 1 "100k" H 2870 2255 50  0000 L CNN
-F 2 "" V 2730 2300 50  0001 C CNN
+F 2 "Resistor_THT:R_Axial_DIN0207_L6.3mm_D2.5mm_P10.16mm_Horizontal" V 2730 2300 50  0001 C CNN
 F 3 "~" H 2800 2300 50  0001 C CNN
 	1    2800 2300
@@
 F 0 "R79" H 2870 2746 50  0000 L CNN
 F 1 "100k" H 2870 2655 50  0000 L CNN
-F 2 "" V 2730 2700 50  0001 C CNN
+F 2 "Resistor_THT:R_Axial_DIN0207_L6.3mm_D2.5mm_P10.16mm_Horizontal" V 2730 2700 50  0001 C CNN
 F 3 "~" H 2800 2700 50  0001 C CNN
 	1    2800 2700
@@
 F 0 "R80" H 3420 2196 50  0000 L CNN
 F 1 "560k" H 3420 2105 50  0000 L CNN
-F 2 "" V 3280 2150 50  0001 C CNN
+F 2 "Resistor_THT:R_Axial_DIN0207_L6.3mm_D2.5mm_P10.16mm_Horizontal" V 3280 2150 50  0001 C CNN
 F 3 "~" H 3350 2150 50  0001 C CNN
 	1    3350 2150
@@
 F 0 "R81" H 3420 2996 50  0000 L CNN
 F 1 "680" H 3420 2905 50  0000 L CNN
-F 2 "" V 3280 2950 50  0001 C CNN
+F 2 "Resistor_THT:R_Axial_DIN0207_L6.3mm_D2.5mm_P10.16mm_Horizontal" V 3280 2950 50  0001 C CNN
 F 3 "~" H 3350 2950 50  0001 C CNN
 	1    3350 2950
@@
 F 0 "R83" H 4870 2796 50  0000 L CNN
 F 1 "10k" H 4870 2705 50  0000 L CNN
-F 2 "" V 4730 2750 50  0001 C CNN
+F 2 "Resistor_THT:R_Axial_DIN0207_L6.3mm_D2.5mm_P10.16mm_Horizontal" V 4730 2750 50  0001 C CNN
 F 3 "~" H 4800 2750 50  0001 C CNN
 	1    4800 2750
@@
 F 0 "R84" H 4870 3146 50  0000 L CNN
 F 1 "4k7" H 4870 3055 50  0000 L CNN
-F 2 "" V 4730 3100 50  0001 C CNN
+F 2 "Resistor_THT:R_Axial_DIN0207_L6.3mm_D2.5mm_P10.16mm_Horizontal" V 4730 3100 50  0001 C CNN
 F 3 "~" H 4800 3100 50  0001 C CNN
 	1    4800 3100
@@
 F 0 "D9" V 5054 3179 50  0000 L CNN
 F 1 "1N4148" V 5145 3179 50  0000 L CNN
-F 2 "" H 5100 3100 50  0001 C CNN
+F 2 "Diode_THT:D_DO-15_P12.70mm_Horizontal" H 5100 3100 50  0001 C CNN
 F 3 "~" H 5100 3100 50  0001 C CNN
 	1    5100 3100
@@
 F 0 "D8" H 5100 2816 50  0000 C CNN
 F 1 "1N4148" H 5100 2725 50  0000 C CNN
-F 2 "" H 5100 2600 50  0001 C CNN
+F 2 "Diode_THT:D_DO-15_P12.70mm_Horizontal" H 5100 2600 50  0001 C CNN
 F 3 "~" H 5100 2600 50  0001 C CNN
 	1    5100 2600
@@
 F 0 "Q16" H 5591 1546 50  0000 L CNN
 F 1 "BF244A" H 5591 1455 50  0000 L CNN
-F 2 "Package_TO_SOT_THT:TO-92_Inline" H 5600 1425 50  0001 L CIN
+F 2 "Package_TO_SOT_THT:TO-92L_Inline_Wide" H 5600 1425 50  0001 L CIN
 F 3 "http://www.fairchildsemi.com/ds/BF/BF244A.pdf" H 5400 1500 50  0001 L CNN
 	1    5400 1500
@@
 F 0 "R82" H 4870 1346 50  0000 L CNN
 F 1 "1k" H 4870 1255 50  0000 L CNN
-F 2 "" V 4730 1300 50  0001 C CNN
+F 2 "Resistor_THT:R_Axial_DIN0207_L6.3mm_D2.5mm_P10.16mm_Horizontal" V 4730 1300 50  0001 C CNN
 F 3 "~" H 4800 1300 50  0001 C CNN
 	1    4800 1300
@@
 F 0 "C14" H 4915 1746 50  0000 L CNN
 F 1 "220nF" H 4915 1655 50  0000 L CNN
-F 2 "" H 4838 1550 50  0001 C CNN
+F 2 "Capacitor_THT:C_Disc_D5.0mm_W2.5mm_P5.00mm" H 4838 1550 50  0001 C CNN
 F 3 "~" H 4800 1700 50  0001 C CNN
 	1    4800 1700
@@
 F 0 "Q17" V 6528 1850 50  0000 C CNN
 F 1 "BF244A" V 6437 1850 50  0000 C CNN
-F 2 "Package_TO_SOT_THT:TO-92_Inline" H 6400 1775 50  0001 L CIN
+F 2 "Package_TO_SOT_THT:TO-92L_Inline_Wide" H 6400 1775 50  0001 L CIN
 F 3 "http://www.fairchildsemi.com/ds/BF/BF244A.pdf" H 6200 1850 50  0001 L CNN
 	1    6200 1850
@@
 F 0 "R85" H 5570 1996 50  0000 L CNN
 F 1 "12k" H 5570 1905 50  0000 L CNN
-F 2 "" V 5430 1950 50  0001 C CNN
+F 2 "Resistor_THT:R_Axial_DIN0207_L6.3mm_D2.5mm_P10.16mm_Horizontal" V 5430 1950 50  0001 C CNN
 F 3 "~" H 5500 1950 50  0001 C CNN
 	1    5500 1950
@@
 F 0 "R86" H 5920 1996 50  0000 L CNN
 F 1 "1M" H 5920 1905 50  0000 L CNN
-F 2 "" V 5780 1950 50  0001 C CNN
+F 2 "Resistor_THT:R_Axial_DIN0207_L6.3mm_D2.5mm_P10.16mm_Horizontal" V 5780 1950 50  0001 C CNN
 F 3 "~" H 5850 1950 50  0001 C CNN
 	1    5850 1950
@@
 F 0 "C15" H 6665 1946 50  0000 L CNN
 F 1 "680nF" H 6665 1855 50  0000 L CNN
-F 2 "" H 6588 1750 50  0001 C CNN
+F 2 "Capacitor_THT:C_Disc_D5.0mm_W2.5mm_P5.00mm" H 6588 1750 50  0001 C CNN
 F 3 "~" H 6550 1900 50  0001 C CNN
 	1    6550 1900
@@
 F 0 "Q18" H 7241 1796 50  0000 L CNN
 F 1 "BF244A" H 7241 1705 50  0000 L CNN
-F 2 "Package_TO_SOT_THT:TO-92_Inline" H 7250 1675 50  0001 L CIN
+F 2 "Package_TO_SOT_THT:TO-92L_Inline_Wide" H 7250 1675 50  0001 L CIN
 F 3 "http://www.fairchildsemi.com/ds/BF/BF244A.pdf" H 7050 1750 50  0001 L CNN
 	1    7050 1750
@@
 F 0 "C17" H 10768 1196 50  0000 L CNN
 F 1 "1uF" H 10768 1105 50  0000 L CNN
-F 2 "" H 10688 1000 50  0001 C CNN
+F 2 "Capacitor_THT:CP_Radial_D6.3mm_P2.50mm" H 10688 1000 50  0001 C CNN
 F 3 "~" H 10650 1150 50  0001 C CNN
 	1    10650 1150
@@
 F 0 "R87" H 7220 2246 50  0000 L CNN
 F 1 "12k" H 7220 2155 50  0000 L CNN
-F 2 "" V 7080 2200 50  0001 C CNN
+F 2 "Resistor_THT:R_Axial_DIN0207_L6.3mm_D2.5mm_P10.16mm_Horizontal" V 7080 2200 50  0001 C CNN
 F 3 "~" H 7150 2200 50  0001 C CNN
 	1    7150 2200
@@
 F 0 "R88" V 7443 2000 50  0000 C CNN
 F 1 "82" V 7534 2000 50  0000 C CNN
-F 2 "" V 7580 2000 50  0001 C CNN
+F 2 "Resistor_THT:R_Axial_DIN0207_L6.3mm_D2.5mm_P10.16mm_Horizontal" V 7580 2000 50  0001 C CNN
 F 3 "~" H 7650 2000 50  0001 C CNN
 	1    7650 2000
@@
 	7150 2000 7150 1950
 $Comp
-L Device:R_POT P9
+L Device:R_POT P7
 U 1 1 5E3A3993
 P 8150 2000
-F 0 "P9" V 8035 2000 50  0000 C CNN
+F 0 "P7" V 8035 2000 50  0000 C CNN
 F 1 "1M" V 7944 2000 50  0000 C CNN
-F 2 "" H 8150 2000 50  0001 C CNN
+F 2 "Connector_PinSocket_2.54mm:PinSocket_1x03_P2.54mm_Vertical" H 8150 2000 50  0001 C CNN
 F 3 "~" H 8150 2000 50  0001 C CNN
+F 4 "GLIDE" V 7850 2000 50  0000 C CNN "Label"
 	1    8150 2000
 	0    -1   -1   0
@@
 F 0 "Q19" H 8791 2046 50  0000 L CNN
 F 1 "BF244A" H 8791 1955 50  0000 L CNN
-F 2 "Package_TO_SOT_THT:TO-92_Inline" H 8800 1925 50  0001 L CIN
+F 2 "Package_TO_SOT_THT:TO-92L_Inline_Wide" H 8800 1925 50  0001 L CIN
 F 3 "http://www.fairchildsemi.com/ds/BF/BF244A.pdf" H 8600 2000 50  0001 L CNN
 	1    8600 2000
@@
 F 0 "R89" H 8770 2546 50  0000 L CNN
 F 1 "12k" H 8770 2455 50  0000 L CNN
-F 2 "" V 8630 2500 50  0001 C CNN
+F 2 "Resistor_THT:R_Axial_DIN0207_L6.3mm_D2.5mm_P10.16mm_Horizontal" V 8630 2500 50  0001 C CNN
 F 3 "~" H 8700 2500 50  0001 C CNN
 	1    8700 2500
@@
 F 0 "R77" H 1670 2246 50  0000 L CNN
 F 1 "31.6" H 1670 2155 50  0000 L CNN
-F 2 "" V 1530 2200 50  0001 C CNN
+F 2 "Resistor_THT:R_Axial_DIN0207_L6.3mm_D2.5mm_P10.16mm_Horizontal" V 1530 2200 50  0001 C CNN
 F 3 "~" H 1600 2200 50  0001 C CNN
 	1    1600 2200
@@
 Connection ~ 2800 2050
 $Comp
-L janel-panel-minimoog-rescue:uA741-DIP14-Amplifier_Operational U8
+L janel-panel-minimoog-rescue:uA741-DIP14-Amplifier_Operational U3
 U 1 1 5E382580
 P 3850 2600
-F 0 "U8" H 3800 2750 50  0000 L CNN
+F 0 "U3" H 3800 2750 50  0000 L CNN
 F 1 "uA741-DIP14" H 3800 2850 50  0000 L CNN
-F 2 "" H 3900 2650 50  0001 C CNN
+F 2 "Package_DIP:DIP-14_W7.62mm_Socket_LongPads" H 3900 2650 50  0001 C CNN
 F 3 "http://www.ti.com/lit/ds/symlink/lm741.pdf" H 4000 2750 50  0001 C CNN
 	1    3850 2600
@@
 F 0 "J1" H 1058 3481 50  0000 C CNN
 F 1 "Conn_01x05_Male" H 1058 3390 50  0000 C CNN
-F 2 "" H 950 3100 50  0001 C CNN
+F 2 "Connector_PinHeader_2.54mm:PinHeader_1x05_P2.54mm_Vertical" H 950 3100 50  0001 C CNN
 F 3 "~" H 950 3100 50  0001 C CNN
 	1    950  3100
