File: LFO.sch (KiCad schematic (older format))
At the start: 16 parts

Commit message: Annotate
Parts:
- gave numbers to parts that had none: 15
Changed lines of the file:
@@
 P 4900 3400
 AR Path="/5E0FCAFC/5E12CD4D" Ref="U?"  Part="1"
-AR Path="/5E124CB8/5E12CD4D" Ref="U?"  Part="1"
-F 0 "U?" H 5244 3446 50  0000 L CNN
+AR Path="/5E124CB8/5E12CD4D" Ref="U1"  Part="1"
+F 0 "U1" H 5244 3446 50  0000 L CNN
 F 1 "UA747" H 5244 3355 50  0000 L CNN
 F 2 "" H 4950 3450 50  0001 C CNN
@@
 P 4150 5150
 AR Path="/5E0FCAFC/5E12CD53" Ref="U?"  Part="2"
-AR Path="/5E124CB8/5E12CD53" Ref="U?"  Part="2"
-F 0 "U?" H 4494 5196 50  0000 L CNN
+AR Path="/5E124CB8/5E12CD53" Ref="U1"  Part="2"
+F 0 "U1" H 4494 5196 50  0000 L CNN
 F 1 "UA747" H 4494 5105 50  0000 L CNN
 F 2 "" H 4200 5200 50  0001 C CNN
@@
 P 7000 3450
 AR Path="/5E0FCAFC/5E12CD6B" Ref="U?"  Part="1"
-AR Path="/5E124CB8/5E12CD6B" Ref="U?"  Part="1"
-F 0 "U?" H 7344 3496 50  0000 L CNN
+AR Path="/5E124CB8/5E12CD6B" Ref="U2"  Part="1"
+F 0 "U2" H 7344 3496 50  0000 L CNN
 F 1 "uA741-DIP14" H 7344 3405 50  0000 L CNN
 F 2 "" H 7050 3500 50  0001 C CNN
@@
 P 5200 4100
 AR Path="/5E0FCAFC/5E12CD7D" Ref="RV?"  Part="1"
-AR Path="/5E124CB8/5E12CD7D" Ref="RV?"  Part="1"
-F 0 "RV?" H 5130 4146 50  0000 R CNN
+AR Path="/5E124CB8/5E12CD7D" Ref="RV1"  Part="1"
+F 0 "RV1" H 5130 4146 50  0000 R CNN
 F 1 "1k" H 5130 4055 50  0000 R CNN
 F 2 "" H 5200 4100 50  0001 C CNN
@@
 P 7150 2900
 AR Path="/5E0FCAFC/5E12CD83" Ref="C?"  Part="1"
-AR Path="/5E124CB8/5E12CD83" Ref="C?"  Part="1"
-F 0 "C?" V 6898 2900 50  0000 C CNN
+AR Path="/5E124CB8/5E12CD83" Ref="C1"  Part="1"
+F 0 "C1" V 6898 2900 50  0000 C CNN
 F 1 "680nF" V 6989 2900 50  0000 C CNN
 F 2 "" H 7188 2750 50  0001 C CNN
@@
 P 6300 4250
 AR Path="/5E0FCAFC/5E12CD89" Ref="R?"  Part="1"
-AR Path="/5E124CB8/5E12CD89" Ref="R?"  Part="1"
-F 0 "R?" V 6093 4250 50  0000 C CNN
+AR Path="/5E124CB8/5E12CD89" Ref="R7"  Part="1"
+F 0 "R7" V 6093 4250 50  0000 C CNN
 F 1 "470" V 6184 4250 50  0000 C CNN
 F 2 "" V 6230 4250 50  0001 C CNN
@@
 P 6300 4550
 AR Path="/5E0FCAFC/5E12CD8F" Ref="R?"  Part="1"
-AR Path="/5E124CB8/5E12CD8F" Ref="R?"  Part="1"
-F 0 "R?" V 6093 4550 50  0000 C CNN
+AR Path="/5E124CB8/5E12CD8F" Ref="R8"  Part="1"
+F 0 "R8" V 6093 4550 50  0000 C CNN
 F 1 "47" V 6184 4550 50  0000 C CNN
 F 2 "" V 6230 4550 50  0001 C CNN
@@
 P 6100 3550
 AR Path="/5E0FCAFC/5E12CD95" Ref="R?"  Part="1"
-AR Path="/5E124CB8/5E12CD95" Ref="R?"  Part="1"
-F 0 "R?" V 5893 3550 50  0000 C CNN
+AR Path="/5E124CB8/5E12CD95" Ref="R6"  Part="1"
+F 0 "R6" V 5893 3550 50  0000 C CNN
 F 1 "68k" V 5984 3550 50  0000 C CNN
 F 2 "" V 6030 3550 50  0001 C CNN
@@
 P 6450 3950
 AR Path="/5E0FCAFC/5E12CD9B" Ref="R?"  Part="1"
-AR Path="/5E124CB8/5E12CD9B" Ref="R?"  Part="1"
-F 0 "R?" H 6520 3996 50  0000 L CNN
+AR Path="/5E124CB8/5E12CD9B" Ref="R9"  Part="1"
+F 0 "R9" H 6520 3996 50  0000 L CNN
 F 1 "68k" H 6520 3905 50  0000 L CNN
 F 2 "" V 6380 3950 50  0001 C CNN
@@
 P 5200 3700
 AR Path="/5E0FCAFC/5E12CDA1" Ref="R?"  Part="1"
-AR Path="/5E124CB8/5E12CDA1" Ref="R?"  Part="1"
-F 0 "R?" H 5270 3746 50  0000 L CNN
+AR Path="/5E124CB8/5E12CDA1" Ref="R3"  Part="1"
+F 0 "R3" H 5270 3746 50  0000 L CNN
 F 1 "3k9" H 5270 3655 50  0000 L CNN
 F 2 "" V 5130 3700 50  0001 C CNN
@@
 P 3650 3650
 AR Path="/5E0FCAFC/5E12CDA7" Ref="R?"  Part="1"
-AR Path="/5E124CB8/5E12CDA7" Ref="R?"  Part="1"
-F 0 "R?" H 3720 3696 50  0000 L CNN
+AR Path="/5E124CB8/5E12CDA7" Ref="R2"  Part="1"
+F 0 "R2" H 3720 3696 50  0000 L CNN
 F 1 "100k" H 3720 3605 50  0000 L CNN
 F 2 "" V 3580 3650 50  0001 C CNN
@@
 P 5650 2600
 AR Path="/5E0FCAFC/5E12CDAD" Ref="R?"  Part="1"
-AR Path="/5E124CB8/5E12CDAD" Ref="R?"  Part="1"
-F 0 "R?" V 5443 2600 50  0000 C CNN
+AR Path="/5E124CB8/5E12CDAD" Ref="R5"  Part="1"
+F 0 "R5" V 5443 2600 50  0000 C CNN
 F 1 "100k" V 5534 2600 50  0000 C CNN
 F 2 "" V 5580 2600 50  0001 C CNN
@@
 P 5650 3550
 AR Path="/5E0FCAFC/5E12CDB3" Ref="P?"  Part="1"
-AR Path="/5E124CB8/5E12CDB3" Ref="P?"  Part="1"
-F 0 "P?" H 5581 3596 50  0000 R CNN
+AR Path="/5E124CB8/5E12CDB3" Ref="P1"  Part="1"
+F 0 "P1" H 5581 3596 50  0000 R CNN
 F 1 "100k" H 5581 3505 50  0000 R CNN
 F 2 "" H 5650 3550 50  0001 C CNN
@@
 P 3600 5250
 AR Path="/5E0FCAFC/5E12CDB9" Ref="R?"  Part="1"
-AR Path="/5E124CB8/5E12CDB9" Ref="R?"  Part="1"
-F 0 "R?" V 3393 5250 50  0000 C CNN
+AR Path="/5E124CB8/5E12CDB9" Ref="R1"  Part="1"
+F 0 "R1" V 3393 5250 50  0000 C CNN
 F 1 "1k" V 3484 5250 50  0000 C CNN
 F 2 "" V 3530 5250 50  0001 C CNN
@@
 P 2950 5150
 AR Path="/5E0FCAFC/5E12CDFC" Ref="K?"  Part="1"
-AR Path="/5E124CB8/5E12CDFC" Ref="K?"  Part="1"
-F 0 "K?" H 2950 5435 50  0000 C CNN
+AR Path="/5E124CB8/5E12CDFC" Ref="K1"  Part="1"
+F 0 "K1" H 2950 5435 50  0000 C CNN
 F 1 "SW_SPDT" H 2950 5344 50  0000 C CNN
 F 2 "" H 2950 5150 50  0001 C CNN
@@
 P 5650 2100
 AR Path="/5E0FCAFC/5E12CE03" Ref="R?"  Part="1"
-AR Path="/5E124CB8/5E12CE03" Ref="R?"  Part="1"
-F 0 "R?" V 5443 2100 50  0000 C CNN
+AR Path="/5E124CB8/5E12CE03" Ref="R4"  Part="1"
+F 0 "R4" V 5443 2100 50  0000 C CNN
 F 1 "1k" V 5534 2100 50  0000 C CNN
 F 2 "" V 5580 2100 50  0001 C CNN

Commit message: VCF work
Parts:
- U1: footprint (none) -> Package_DIP:DIP-14_W7.62mm_LongPads; symbol Amplifier_Operational:UA747 -> janel-panel-minimoog-rescue:UA747-Amplifier_Operational
- U2: footprint (none) -> Package_DIP:DIP-14_W7.62mm_LongPads; symbol Amplifier_Operational:uA741-DIP14 -> Amplifier_Operational:LM741
Changed lines of the file:
@@
 $EndDescr
 $Comp
-L Amplifier_Operational:UA747 U?
+L janel-panel-minimoog-rescue:UA747-Amplifier_Operational U?
 U 1 1 5E12CD4D
 P 4900 3400
 AR Path="/5E0FCAFC/5E12CD4D" Ref="U?"  Part="1"
 AR Path="/5E124CB8/5E12CD4D" Ref="U1"  Part="1"
+AR Path="/5E12CD4D" Ref="U1"  Part="1"
 F 0 "U1" H 5244 3446 50  0000 L CNN
 F 1 "UA747" H 5244 3355 50  0000 L CNN
-F 2 "" H 4950 3450 50  0001 C CNN
+F 2 "Package_DIP:DIP-14_W7.62mm_LongPads" H 4950 3450 50  0001 C CNN
 F 3 "https://www.ti.com/lit/ds/symlink/ua747.pdf" H 5050 3550 50  0001 C CNN
 	1    4900 3400
@@
 $EndComp
 $Comp
-L Amplifier_Operational:UA747 U?
+L janel-panel-minimoog-rescue:UA747-Amplifier_Operational U?
 U 2 1 5E12CD53
 P 4150 5150
 AR Path="/5E0FCAFC/5E12CD53" Ref="U?"  Part="2"
 AR Path="/5E124CB8/5E12CD53" Ref="U1"  Part="2"
+AR Path="/5E12CD53" Ref="U1"  Part="2"
 F 0 "U1" H 4494 5196 50  0000 L CNN
 F 1 "UA747" H 4494 5105 50  0000 L CNN
-F 2 "" H 4200 5200 50  0001 C CNN
+F 2 "Package_DIP:DIP-14_W7.62mm_LongPads" H 4200 5200 50  0001 C CNN
 F 3 "https://www.ti.com/lit/ds/symlink/ua747.pdf" H 4300 5300 50  0001 C CNN
 	2    4150 5150
@@
 $EndComp
 $Comp
-L Amplifier_Operational:uA741-DIP14 U?
+L Amplifier_Operational:LM741 U?
 U 1 1 5E12CD6B
 P 7000 3450
@@
 F 0 "U2" H 7344 3496 50  0000 L CNN
 F 1 "uA741-DIP14" H 7344 3405 50  0000 L CNN
-F 2 "" H 7050 3500 50  0001 C CNN
+F 2 "Package_DIP:DIP-14_W7.62mm_LongPads" H 7050 3500 50  0001 C CNN
 F 3 "http://www.ti.com/lit/ds/symlink/lm741.pdf" H 7150 3600 50  0001 C CNN
 	1    7000 3450

Commit message: Update some components
Parts:
- renumbered C1 to C5, R4 to R10, R5 to R11, R6 to R12, R7 to R13, R8 to R14, R9 to R15, R1 to R7, R2 to R8, R3 to R9, RV1 to RV2
Connections:
- no-connect marks 6 -> 2
Changed lines of the file:
@@
 AR Path="/5E0FCAFC/5E12CD4D" Ref="U?"  Part="1"
 AR Path="/5E124CB8/5E12CD4D" Ref="U1"  Part="1"
-AR Path="/5E12CD4D" Ref="U1"  Part="1"
+AR Path="/5E12CD4D" Ref="U?"  Part="1"
 F 0 "U1" H 5244 3446 50  0000 L CNN
 F 1 "UA747" H 5244 3355 50  0000 L CNN
@@
 AR Path="/5E0FCAFC/5E12CD53" Ref="U?"  Part="2"
 AR Path="/5E124CB8/5E12CD53" Ref="U1"  Part="2"
-AR Path="/5E12CD53" Ref="U1"  Part="2"
+AR Path="/5E12CD53" Ref="U?"  Part="2"
 F 0 "U1" H 4494 5196 50  0000 L CNN
 F 1 "UA747" H 4494 5105 50  0000 L CNN
@@
 P 4800 3100
 AR Path="/5E0FCAFC/5E12CD59" Ref="#PWR?"  Part="1"
-AR Path="/5E124CB8/5E12CD59" Ref="#PWR0107"  Part="1"
-F 0 "#PWR0107" H 4800 2950 50  0001 C CNN
+AR Path="/5E124CB8/5E12CD59" Ref="#PWR011"  Part="1"
+F 0 "#PWR011" H 4800 2950 50  0001 C CNN
 F 1 "+VSW" H 4815 3273 50  0000 C CNN
 F 2 "" H 4800 3100 50  0001 C CNN
@@
 P 4800 3700
 AR Path="/5E0FCAFC/5E12CD5F" Ref="#PWR?"  Part="1"
-AR Path="/5E124CB8/5E12CD5F" Ref="#PWR0108"  Part="1"
-F 0 "#PWR0108" H 4800 3800 50  0001 C CNN
+AR Path="/5E124CB8/5E12CD5F" Ref="#PWR012"  Part="1"
+F 0 "#PWR012" H 4800 3800 50  0001 C CNN
 F 1 "-VSW" H 4815 3873 50  0000 C CNN
 F 2 "" H 4800 3700 50  0001 C CNN
@@
 P 6900 3750
 AR Path="/5E0FCAFC/5E12CD65" Ref="#PWR?"  Part="1"
-AR Path="/5E124CB8/5E12CD65" Ref="#PWR0109"  Part="1"
-F 0 "#PWR0109" H 6900 3850 50  0001 C CNN
+AR Path="/5E124CB8/5E12CD65" Ref="#PWR015"  Part="1"
+F 0 "#PWR015" H 6900 3850 50  0001 C CNN
 F 1 "-VSW" H 6915 3923 50  0000 C CNN
 F 2 "" H 6900 3750 50  0001 C CNN
@@
 P 6900 3150
 AR Path="/5E0FCAFC/5E12CD71" Ref="#PWR?"  Part="1"
-AR Path="/5E124CB8/5E12CD71" Ref="#PWR0110"  Part="1"
-F 0 "#PWR0110" H 6900 3000 50  0001 C CNN
+AR Path="/5E124CB8/5E12CD71" Ref="#PWR014"  Part="1"
+F 0 "#PWR014" H 6900 3000 50  0001 C CNN
 F 1 "+VSW" H 6915 3323 50  0000 C CNN
 F 2 "" H 6900 3150 50  0001 C CNN
@@
 P 4050 4850
 AR Path="/5E0FCAFC/5E12CD77" Ref="#PWR?"  Part="1"
-AR Path="/5E124CB8/5E12CD77" Ref="#PWR0111"  Part="1"
-F 0 "#PWR0111" H 4050 4700 50  0001 C CNN
+AR Path="/5E124CB8/5E12CD77" Ref="#PWR09"  Part="1"
+F 0 "#PWR09" H 4050 4700 50  0001 C CNN
 F 1 "+VSW" H 4065 5023 50  0000 C CNN
 F 2 "" H 4050 4850 50  0001 C CNN
@@
 P 5200 4100
 AR Path="/5E0FCAFC/5E12CD7D" Ref="RV?"  Part="1"
-AR Path="/5E124CB8/5E12CD7D" Ref="RV1"  Part="1"
-F 0 "RV1" H 5130 4146 50  0000 R CNN
+AR Path="/5E124CB8/5E12CD7D" Ref="RV2"  Part="1"
+F 0 "RV2" H 5130 4146 50  0000 R CNN
 F 1 "1k" H 5130 4055 50  0000 R CNN
 F 2 "" H 5200 4100 50  0001 C CNN
@@
 P 7150 2900
 AR Path="/5E0FCAFC/5E12CD83" Ref="C?"  Part="1"
-AR Path="/5E124CB8/5E12CD83" Ref="C1"  Part="1"
-F 0 "C1" V 6898 2900 50  0000 C CNN
+AR Path="/5E124CB8/5E12CD83" Ref="C5"  Part="1"
+F 0 "C5" V 6898 2900 50  0000 C CNN
 F 1 "680nF" V 6989 2900 50  0000 C CNN
 F 2 "" H 7188 2750 50  0001 C CNN
@@
 P 6300 4250
 AR Path="/5E0FCAFC/5E12CD89" Ref="R?"  Part="1"
-AR Path="/5E124CB8/5E12CD89" Ref="R7"  Part="1"
-F 0 "R7" V 6093 4250 50  0000 C CNN
+AR Path="/5E124CB8/5E12CD89" Ref="R13"  Part="1"
+F 0 "R13" V 6093 4250 50  0000 C CNN
 F 1 "470" V 6184 4250 50  0000 C CNN
 F 2 "" V 6230 4250 50  0001 C CNN
@@
 P 6300 4550
 AR Path="/5E0FCAFC/5E12CD8F" Ref="R?"  Part="1"
-AR Path="/5E124CB8/5E12CD8F" Ref="R8"  Part="1"
-F 0 "R8" V 6093 4550 50  0000 C CNN
+AR Path="/5E124CB8/5E12CD8F" Ref="R14"  Part="1"
+F 0 "R14" V 6093 4550 50  0000 C CNN
 F 1 "47" V 6184 4550 50  0000 C CNN
 F 2 "" V 6230 4550 50  0001 C CNN
@@
 P 6100 3550
 AR Path="/5E0FCAFC/5E12CD95" Ref="R?"  Part="1"
-AR Path="/5E124CB8/5E12CD95" Ref="R6"  Part="1"
-F 0 "R6" V 5893 3550 50  0000 C CNN
+AR Path="/5E124CB8/5E12CD95" Ref="R12"  Part="1"
+F 0 "R12" V 5893 3550 50  0000 C CNN
 F 1 "68k" V 5984 3550 50  0000 C CNN
 F 2 "" V 6030 3550 50  0001 C CNN
@@
 P 6450 3950
 AR Path="/5E0FCAFC/5E12CD9B" Ref="R?"  Part="1"
-AR Path="/5E124CB8/5E12CD9B" Ref="R9"  Part="1"
-F 0 "R9" H 6520 3996 50  0000 L CNN
+AR Path="/5E124CB8/5E12CD9B" Ref="R15"  Part="1"
+F 0 "R15" H 6520 3996 50  0000 L CNN
 F 1 "68k" H 6520 3905 50  0000 L CNN
 F 2 "" V 6380 3950 50  0001 C CNN
@@
 P 5200 3700
 AR Path="/5E0FCAFC/5E12CDA1" Ref="R?"  Part="1"
-AR Path="/5E124CB8/5E12CDA1" Ref="R3"  Part="1"
-F 0 "R3" H 5270 3746 50  0000 L CNN
+AR Path="/5E124CB8/5E12CDA1" Ref="R9"  Part="1"
+F 0 "R9" H 5270 3746 50  0000 L CNN
 F 1 "3k9" H 5270 3655 50  0000 L CNN
 F 2 "" V 5130 3700 50  0001 C CNN
@@
 P 3650 3650
 AR Path="/5E0FCAFC/5E12CDA7" Ref="R?"  Part="1"
-AR Path="/5E124CB8/5E12CDA7" Ref="R2"  Part="1"
-F 0 "R2" H 3720 3696 50  0000 L CNN
+AR Path="/5E124CB8/5E12CDA7" Ref="R8"  Part="1"
+F 0 "R8" H 3720 3696 50  0000 L CNN
 F 1 "100k" H 3720 3605 50  0000 L CNN
 F 2 "" V 3580 3650 50  0001 C CNN
@@
 P 5650 2600
 AR Path="/5E0FCAFC/5E12CDAD" Ref="R?"  Part="1"
-AR Path="/5E124CB8/5E12CDAD" Ref="R5"  Part="1"
-F 0 "R5" V 5443 2600 50  0000 C CNN
+AR Path="/5E124CB8/5E12CDAD" Ref="R11"  Part="1"
+F 0 "R11" V 5443 2600 50  0000 C CNN
 F 1 "100k" V 5534 2600 50  0000 C CNN
 F 2 "" V 5580 2600 50  0001 C CNN
@@
 P 3600 5250
 AR Path="/5E0FCAFC/5E12CDB9" Ref="R?"  Part="1"
-AR Path="/5E124CB8/5E12CDB9" Ref="R1"  Part="1"
-F 0 "R1" V 3393 5250 50  0000 C CNN
+AR Path="/5E124CB8/5E12CDB9" Ref="R7"  Part="1"
+F 0 "R7" V 3393 5250 50  0000 C CNN
 F 1 "1k" V 3484 5250 50  0000 C CNN
 F 2 "" V 3530 5250 50  0001 C CNN
@@
 P 4500 3650
 AR Path="/5E0FCAFC/5E12CDBF" Ref="#PWR?"  Part="1"
-AR Path="/5E124CB8/5E12CDBF" Ref="#PWR0112"  Part="1"
-F 0 "#PWR0112" H 4500 3400 50  0001 C CNN
+AR Path="/5E124CB8/5E12CDBF" Ref="#PWR010"  Part="1"
+F 0 "#PWR010" H 4500 3400 50  0001 C CNN
 F 1 "GND" H 4505 3477 50  0000 C CNN
 F 2 "" H 4500 3650 50  0001 C CNN
@@
 Wire Wire Line
 	3800 5250 3750 5250
-NoConn ~ 4150 5450
-NoConn ~ 4250 5450
 Wire Wire Line
 	4500 3650 4500 3500
@@
 P 6450 4750
 AR Path="/5E0FCAFC/5E12CDDD" Ref="#PWR?"  Part="1"
-AR Path="/5E124CB8/5E12CDDD" Ref="#PWR0113"  Part="1"
-F 0 "#PWR0113" H 6450 4500 50  0001 C CNN
+AR Path="/5E124CB8/5E12CDDD" Ref="#PWR013"  Part="1"
+F 0 "#PWR013" H 6450 4500 50  0001 C CNN
 F 1 "GND" H 6455 4577 50  0000 C CNN
 F 2 "" H 6450 4750 50  0001 C CNN
@@
 Wire Wire Line
 	5200 3400 5200 3550
-NoConn ~ 4900 3700
-NoConn ~ 5000 3700
 Wire Wire Line
 	5650 3700 5650 4550
@@
 P 5650 2100
 AR Path="/5E0FCAFC/5E12CE03" Ref="R?"  Part="1"
-AR Path="/5E124CB8/5E12CE03" Ref="R4"  Part="1"
-F 0 "R4" V 5443 2100 50  0000 C CNN
+AR Path="/5E124CB8/5E12CE03" Ref="R10"  Part="1"
+F 0 "R10" V 5443 2100 50  0000 C CNN
 F 1 "1k" V 5534 2100 50  0000 C CNN
 F 2 "" V 5580 2100 50  0001 C CNN

Commit message: Create pcb and other updates
Parts:
- C5: footprint (none) -> Capacitor_THT:C_Disc_D5.0mm_W2.5mm_P5.00mm
- K4: renamed from K1; footprint (none) -> Connector_PinSocket_2.54mm:PinSocket_1x03_P2.54mm_Vertical
- P1: footprint (none) -> Connector_PinSocket_2.54mm:PinSocket_1x03_P2.54mm_Vertical
- R10, R11, R12, R13, R14, R15, R7, R8, R9: footprint (none) -> Resistor_THT:R_Axial_DIN0207_L6.3mm_D2.5mm_P10.16mm_Horizontal
- RV2: footprint (none) -> Potentiometer_THT:Potentiometer_Bourns_3296W_Vertical
- U5: renamed from U2; footprint Package_DIP:DIP-14_W7.62mm_LongPads -> Package_DIP:DIP-14_W7.62mm_Socket_LongPads
- U6: renamed from U1; footprint Package_DIP:DIP-14_W7.62mm_LongPads -> Package_DIP:DIP-14_W7.62mm_Socket_LongPads
Changed lines of the file:
@@
 P 4900 3400
 AR Path="/5E0FCAFC/5E12CD4D" Ref="U?"  Part="1"
-AR Path="/5E124CB8/5E12CD4D" Ref="U1"  Part="1"
+AR Path="/5E124CB8/5E12CD4D" Ref="U6"  Part="1"
 AR Path="/5E12CD4D" Ref="U?"  Part="1"
-F 0 "U1" H 5244 3446 50  0000 L CNN
+F 0 "U6" H 5244 3446 50  0000 L CNN
 F 1 "UA747" H 5244 3355 50  0000 L CNN
-F 2 "Package_DIP:DIP-14_W7.62mm_LongPads" H 4950 3450 50  0001 C CNN
+F 2 "Package_DIP:DIP-14_W7.62mm_Socket_LongPads" H 4950 3450 50  0001 C CNN
 F 3 "https://www.ti.com/lit/ds/symlink/ua747.pdf" H 5050 3550 50  0001 C CNN
 	1    4900 3400
@@
 P 4150 5150
 AR Path="/5E0FCAFC/5E12CD53" Ref="U?"  Part="2"
-AR Path="/5E124CB8/5E12CD53" Ref="U1"  Part="2"
+AR Path="/5E124CB8/5E12CD53" Ref="U6"  Part="2"
 AR Path="/5E12CD53" Ref="U?"  Part="2"
-F 0 "U1" H 4494 5196 50  0000 L CNN
+F 0 "U6" H 4494 5196 50  0000 L CNN
 F 1 "UA747" H 4494 5105 50  0000 L CNN
-F 2 "Package_DIP:DIP-14_W7.62mm_LongPads" H 4200 5200 50  0001 C CNN
+F 2 "Package_DIP:DIP-14_W7.62mm_Socket_LongPads" H 4200 5200 50  0001 C CNN
 F 3 "https://www.ti.com/lit/ds/symlink/ua747.pdf" H 4300 5300 50  0001 C CNN
 	2    4150 5150
@@
 P 7000 3450
 AR Path="/5E0FCAFC/5E12CD6B" Ref="U?"  Part="1"
-AR Path="/5E124CB8/5E12CD6B" Ref="U2"  Part="1"
-F 0 "U2" H 7344 3496 50  0000 L CNN
+AR Path="/5E124CB8/5E12CD6B" Ref="U5"  Part="1"
+F 0 "U5" H 7344 3496 50  0000 L CNN
 F 1 "uA741-DIP14" H 7344 3405 50  0000 L CNN
-F 2 "Package_DIP:DIP-14_W7.62mm_LongPads" H 7050 3500 50  0001 C CNN
+F 2 "Package_DIP:DIP-14_W7.62mm_Socket_LongPads" H 7050 3500 50  0001 C CNN
 F 3 "http://www.ti.com/lit/ds/symlink/lm741.pdf" H 7150 3600 50  0001 C CNN
 	1    7000 3450
@@
 F 0 "RV2" H 5130 4146 50  0000 R CNN
 F 1 "1k" H 5130 4055 50  0000 R CNN
-F 2 "" H 5200 4100 50  0001 C CNN
+F 2 "Potentiometer_THT:Potentiometer_Bourns_3296W_Vertical" H 5200 4100 50  0001 C CNN
 F 3 "~" H 5200 4100 50  0001 C CNN
 	1    5200 4100
@@
 F 0 "C5" V 6898 2900 50  0000 C CNN
 F 1 "680nF" V 6989 2900 50  0000 C CNN
-F 2 "" H 7188 2750 50  0001 C CNN
+F 2 "Capacitor_THT:C_Disc_D5.0mm_W2.5mm_P5.00mm" H 7188 2750 50  0001 C CNN
 F 3 "~" H 7150 2900 50  0001 C CNN
 	1    7150 2900
@@
 F 0 "R13" V 6093 4250 50  0000 C CNN
 F 1 "470" V 6184 4250 50  0000 C CNN
-F 2 "" V 6230 4250 50  0001 C CNN
+F 2 "Resistor_THT:R_Axial_DIN0207_L6.3mm_D2.5mm_P10.16mm_Horizontal" V 6230 4250 50  0001 C CNN
 F 3 "~" H 6300 4250 50  0001 C CNN
 	1    6300 4250
@@
 F 0 "R14" V 6093 4550 50  0000 C CNN
 F 1 "47" V 6184 4550 50  0000 C CNN
-F 2 "" V 6230 4550 50  0001 C CNN
+F 2 "Resistor_THT:R_Axial_DIN0207_L6.3mm_D2.5mm_P10.16mm_Horizontal" V 6230 4550 50  0001 C CNN
 F 3 "~" H 6300 4550 50  0001 C CNN
 	1    6300 4550
@@
 F 0 "R12" V 5893 3550 50  0000 C CNN
 F 1 "68k" V 5984 3550 50  0000 C CNN
-F 2 "" V 6030 3550 50  0001 C CNN
+F 2 "Resistor_THT:R_Axial_DIN0207_L6.3mm_D2.5mm_P10.16mm_Horizontal" V 6030 3550 50  0001 C CNN
 F 3 "~" H 6100 3550 50  0001 C CNN
 	1    6100 3550
@@
 F 0 "R15" H 6520 3996 50  0000 L CNN
 F 1 "68k" H 6520 3905 50  0000 L CNN
-F 2 "" V 6380 3950 50  0001 C CNN
+F 2 "Resistor_THT:R_Axial_DIN0207_L6.3mm_D2.5mm_P10.16mm_Horizontal" V 6380 3950 50  0001 C CNN
 F 3 "~" H 6450 3950 50  0001 C CNN
 	1    6450 3950
@@
 F 0 "R9" H 5270 3746 50  0000 L CNN
 F 1 "3k9" H 5270 3655 50  0000 L CNN
-F 2 "" V 5130 3700 50  0001 C CNN
+F 2 "Resistor_THT:R_Axial_DIN0207_L6.3mm_D2.5mm_P10.16mm_Horizontal" V 5130 3700 50  0001 C CNN
 F 3 "~" H 5200 3700 50  0001 C CNN
 	1    5200 3700
@@
 F 0 "R8" H 3720 3696 50  0000 L CNN
 F 1 "100k" H 3720 3605 50  0000 L CNN
-F 2 "" V 3580 3650 50  0001 C CNN
+F 2 "Resistor_THT:R_Axial_DIN0207_L6.3mm_D2.5mm_P10.16mm_Horizontal" V 3580 3650 50  0001 C CNN
 F 3 "~" H 3650 3650 50  0001 C CNN
 	1    3650 3650
@@
 F 0 "R11" V 5443 2600 50  0000 C CNN
 F 1 "100k" V 5534 2600 50  0000 C CNN
-F 2 "" V 5580 2600 50  0001 C CNN
+F 2 "Resistor_THT:R_Axial_DIN0207_L6.3mm_D2.5mm_P10.16mm_Horizontal" V 5580 2600 50  0001 C CNN
 F 3 "~" H 5650 2600 50  0001 C CNN
 	1    5650 2600
@@
 F 0 "P1" H 5581 3596 50  0000 R CNN
 F 1 "100k" H 5581 3505 50  0000 R CNN
-F 2 "" H 5650 3550 50  0001 C CNN
+F 2 "Connector_PinSocket_2.54mm:PinSocket_1x03_P2.54mm_Vertical" H 5650 3550 50  0001 C CNN
 F 3 "~" H 5650 3550 50  0001 C CNN
 	1    5650 3550
@@
 F 0 "R7" V 3393 5250 50  0000 C CNN
 F 1 "1k" V 3484 5250 50  0000 C CNN
-F 2 "" V 3530 5250 50  0001 C CNN
+F 2 "Resistor_THT:R_Axial_DIN0207_L6.3mm_D2.5mm_P10.16mm_Horizontal" V 3530 5250 50  0001 C CNN
 F 3 "~" H 3600 5250 50  0001 C CNN
 	1    3600 5250
@@
 P 2950 5150
 AR Path="/5E0FCAFC/5E12CDFC" Ref="K?"  Part="1"
-AR Path="/5E124CB8/5E12CDFC" Ref="K1"  Part="1"
-F 0 "K1" H 2950 5435 50  0000 C CNN
+AR Path="/5E124CB8/5E12CDFC" Ref="K4"  Part="1"
+F 0 "K4" H 2950 5435 50  0000 C CNN
 F 1 "SW_SPDT" H 2950 5344 50  0000 C CNN
-F 2 "" H 2950 5150 50  0001 C CNN
+F 2 "Connector_PinSocket_2.54mm:PinSocket_1x03_P2.54mm_Vertical" H 2950 5150 50  0001 C CNN
 F 3 "~" H 2950 5150 50  0001 C CNN
 	1    2950 5150
@@
 F 0 "R10" V 5443 2100 50  0000 C CNN
 F 1 "1k" V 5534 2100 50  0000 C CNN
-F 2 "" V 5580 2100 50  0001 C CNN
+F 2 "Resistor_THT:R_Axial_DIN0207_L6.3mm_D2.5mm_P10.16mm_Horizontal" V 5580 2100 50  0001 C CNN
 F 3 "~" H 5650 2100 50  0001 C CNN
 	1    5650 2100
