File: VCF.sch (KiCad schematic (older format))
At the start: 10 parts, among them U10 UA747, U12 CA3080A, U13 CA3080A, U8 UA747, U9 CA3080A

Commit message: VCF work
Parts:
- added C? (x2): 1nF, symbol Device:C
- added C?: 680nF, symbol Device:C
- added Q? (x3): Q_PNP_BCE, symbol Device:Q_PNP_BCE
- added Q?: Q_BC_214_PNP, symbol Device:Q_PNP_BCE
- added R? (x2): 330k, symbol Device:R
- added R? (x3): 2k2, symbol Device:R
- added R? (x2): 27k, symbol Device:R
- added R?: 330, symbol Device:R
- added R? (x3): 100k, symbol Device:R
- added R?: 33k, symbol Device:R
- added R?: 47k, symbol Device:R
- added RV? (x2): 100k, symbol Device:R_POT
- added RV? (x2): 50k, symbol Device:R_POT
- added SW?: SW_SPST, symbol Switch:SW_SPST
Connections:
- net labels added: CV, ENVELOPE
- wire segments 10 -> 65
- no-connect marks 4 -> 8
Other:
- moved on the sheet: U12, U13, U9

Commit message: VCF work
Parts:
- added C? (x2): 220pF, symbol Device:C_Small
- added C?: 33pF, symbol Device:C_Small
- added Q? (x2): BF244A, Package_TO_SOT_THT:TO-92_Inline, symbol Transistor_FET:BF244A
- added R? (x6): 100, symbol Device:R
- added R? (x2): 12k, symbol Device:R
- added R?: 330k, symbol Device:R
- added R? (x3): 39k, symbol Device:R
- added R? (x3): 100k, symbol Device:R
- added R?: 27k, symbol Device:R
- added R?: 330, symbol Device:R
- added RV?: 100k, symbol Device:R_POT_TRIM
- added SW10, SW8, SW9: SW_SPST, symbol Switch:SW_SPST
- R?: value R -> 10k
- U10, U8: symbol Amplifier_Operational:UA747 -> janel-panel-minimoog-rescue:UA747-Amplifier_Operational
Connections:
- net labels added: Ivca_cv, Ivcf_cv, TO_VCA
- wire segments 65 -> 119
- no-connect marks 8 -> 6
Other:
- moved on the sheet: C?, Q?, R?, RV?, SW?, U12, U13, U9

Commit message: VCF finished
Parts:
- added C?: 4.7uF, symbol Device:CP_Small
- added C?: 33nF, symbol Device:C_Small
- added P12, P14: 100k, symbol Device:R_POT
- added P13: 22k, symbol Device:R_POT
- added Q?: Q_NPN_BCE, symbol Device:Q_NPN_BCE
- added R9: 100k, symbol Device:R_POT_TRIM
- added R? (x2): 100k, symbol Device:R
- added R?: 47k, symbol Device:R
- added R?: 51k, symbol Device:R
- added R?: 1M, symbol Device:R
- added R?: 12k, symbol Device:R
- added R?: 22k, symbol Device:R
- added R? (x2): 1k, symbol Device:R
- added R?: 39k, symbol Device:R
- R?: value 330 -> 330k
- gave numbers to parts that had none: 5
Connections:
- net +VSW: now also U10.9 (V+), Q?.2 (C), R?.1
- net -VSW: now also R8.3, R?.1, R?.1, R9.1, R?.2
- net 5V?: now also R?.1
- net ENVELOPE: now also R?.1
- net GND: now also R?.2, P13.1, P14.3, R9.3, R?.1, R?.1
- net at U13.6: now also Q?.1 (B), R?.2
- net at R?.1, R?.2, U8.1 (-): now also C?.2, R?.2, R?.2
- net at Q?.1 (B): now also P14.1, R?.1, R?.2, R?.2
- net at Q?.3 (S), R?.2, SW8.2 (B): now also C?.1, R?.1
- net at R?.1, SW9.2 (B): now also P12.1
- new net: R9.2, R?.2
- new net: P14.2, R?.2
- new net: C?.1, Q?.3 (E), R?.1
- new net: P13.3, R?.1
- new net: C?.2, R?.2
- new net: P12.2, R?.1
- new net: P12.3, R?.2
- new net OUTPUT: P13.2
- no-connect marks 6 -> 0

Commit message: Update some components
Parts:
- gave numbers to parts that had none: 61
- renumbered P8 to P10, P9 to P11, P10 to P12, P11 to P13, P12 to P14, P14 to P15, P13 to P16, R9 to R115, R8 to R133, SW10 to SW3, SW9 to SW4, SW8 to SW5, U8 to U11

Commit message: ERC pass
Parts:
- added JP1: Jumper_NO_Small, symbol Device:Jumper_NO_Small
Connections:
- net GND: now also JP1.2
- net OUTPUT: now also JP1.1
Changed lines of the file:
@@
 Wire Wire Line
 	10350 2750 10550 2750
+$Comp
+L Device:Jumper_NO_Small JP1
+U 1 1 5E9D1FA7
+P 10800 2900
+F 0 "JP1" H 10800 3085 50  0000 C CNN
+F 1 "Jumper_NO_Small" H 10800 2994 50  0000 C CNN
+F 2 "" H 10800 2900 50  0001 C CNN
+F 3 "~" H 10800 2900 50  0001 C CNN
+	1    10800 2900
+	1    0    0    -1
+$EndComp
+$Comp
+L power:GND #PWR0128
+U 1 1 5E9D2A41
+P 10900 2900
+F 0 "#PWR0128" H 10900 2650 50  0001 C CNN
+F 1 "GND" H 10905 2727 50  0000 C CNN
+F 2 "" H 10900 2900 50  0001 C CNN
+F 3 "" H 10900 2900 50  0001 C CNN
+	1    10900 2900
+	1    0    0    -1
+$EndComp
 $EndSCHEMATC

Commit message: Create pcb and other updates
Parts:
- C18, C19, C20, C21, C22, C23, C24: footprint (none) -> Capacitor_THT:C_Disc_D5.0mm_W2.5mm_P5.00mm
- C25: footprint (none) -> Capacitor_THT:CP_Radial_D6.3mm_P2.50mm
- JP1: footprint (none) -> Connector_PinHeader_2.54mm:PinHeader_1x02_P2.54mm_Vertical
- K10: renamed from SW3; footprint (none) -> Connector_PinSocket_2.54mm:PinSocket_1x03_P2.54mm_Vertical
- K7: renamed from SW2; footprint (none) -> Connector_PinSocket_2.54mm:PinSocket_1x03_P2.54mm_Vertical
- K8: renamed from SW5; footprint (none) -> Connector_PinSocket_2.54mm:PinSocket_1x03_P2.54mm_Vertical
- K9: renamed from SW4; footprint (none) -> Connector_PinSocket_2.54mm:PinSocket_1x03_P2.54mm_Vertical
- P10: renamed from P12; footprint (none) -> Connector_PinSocket_2.54mm:PinSocket_1x03_P2.54mm_Vertical
- P11: renamed from P13; footprint (none) -> Connector_PinSocket_2.54mm:PinSocket_1x03_P2.54mm_Vertical
- P12: renamed from P14; footprint (none) -> Connector_PinSocket_2.54mm:PinSocket_1x03_P2.54mm_Vertical
- P14: renamed from P15; footprint (none) -> Connector_PinSocket_2.54mm:PinSocket_1x03_P2.54mm_Vertical
- P16: footprint (none) -> Connector_PinSocket_2.54mm:PinSocket_1x03_P2.54mm_Vertical
- P8: renamed from P10; footprint (none) -> Connector_PinSocket_2.54mm:PinSocket_1x03_P2.54mm_Vertical
- P9: renamed from P11; footprint (none) -> Connector_PinSocket_2.54mm:PinSocket_1x03_P2.54mm_Vertical
- Q20, Q23: footprint Package_TO_SOT_THT:TO-92_Inline -> Package_TO_SOT_THT:TO-92L_Inline_Wide
- Q21, Q22, Q24, Q25, Q26: footprint (none) -> Package_TO_SOT_THT:TO-92L_Inline_Wide
- R100, R101, R102, R103, R104, R105, R106, R107, R108, R109, R110, R111, R112, R113, R114, R116, R117, R118, R119, R120, R121, R122, R123, R124, R125, R126, R127, R128, R129, R130, R131, R132, R134, R135, R136, R90, R91, R92, R93, R94, R95, R96, R97, R98, R99: footprint (none) -> Resistor_THT:R_Axial_DIN0207_L6.3mm_D2.5mm_P10.16mm_Horizontal
- RV133: renamed from R133; footprint (none) -> Potentiometer_THT:Potentiometer_Bourns_3296W_Vertical
- RV9_1: renamed from R115; footprint (none) -> Potentiometer_THT:Potentiometer_Bourns_3296W_Vertical
- U10: footprint (none) -> Package_DIP:DIP-14_W7.62mm_Socket_LongPads
- U12, U13, U9: footprint (none) -> Package_DIP:DIP-8_W7.62mm_Socket_LongPads
- U8: renamed from U11; footprint (none) -> Package_DIP:DIP-14_W7.62mm_Socket_LongPads
Connections:
- net 5V? renamed LFO_OUT
- net LFO_OUT: no longer R90.2
- new net TO_VCF: R90.2
Other:
- moved on the sheet: Q22
