File: VCO.sch (KiCad schematic (older format))
At the start: 57 parts, among them K1 SW_SPST, K2 SW_SPST, K3 SW_SPST, P2 100k, P3 100k, P4 4k7, U1 7413, U2 7490

Commit message: Annotate
Parts:
- gave numbers to parts that had none: 45

Commit message: VCF work
Parts:
- U3: symbol Amplifier_Operational:UA747 -> janel-panel-minimoog-rescue:UA747-Amplifier_Operational
Changed lines of the file:
@@
 	6700 5250 6700 5100
 $Comp
-L Amplifier_Operational:UA747 U3
+L janel-panel-minimoog-rescue:UA747-Amplifier_Operational U3
 U 1 1 5E216D73
 P 6350 5800
+AR Path="/5E216D73" Ref="U3"  Part="1"
+AR Path="/5E12E25C/5E216D73" Ref="U3"  Part="1"
 F 0 "U3" H 6694 5846 50  0000 L CNN
 F 1 "UA747" H 6694 5755 50  0000 L CNN
@@
 $EndComp
 $Comp
-L Amplifier_Operational:UA747 U3
+L janel-panel-minimoog-rescue:UA747-Amplifier_Operational U3
 U 2 1 5E217D9A
 P 8500 5900
+AR Path="/5E217D9A" Ref="U3"  Part="2"
+AR Path="/5E12E25C/5E217D9A" Ref="U3"  Part="2"
 F 0 "U3" H 8844 5946 50  0000 L CNN
 F 1 "UA747" H 8844 5855 50  0000 L CNN

Commit message: Update some components
Parts:
- renumbered C5 to C10, C6 to C11, C1 to C6, C2 to C7, C3 to C8, C4 to C9, K3 to K2, K2 to K3, K1 to K4, P3 to P2, P2 to P3, Q1 to Q3, Q2 to Q4, Q3 to Q5, Q4 to Q6, Q5 to Q7, Q6 to Q8, R2 to R16, R4 to R17, R1 to R18, R3 to R19, R6 to R20, R7 to R21, R8 to R22, R9 to R23, R10 to R24, R11 to R25, R12 to R26, R13 to R27, R14 to R28, R15 to R29, R16 to R30, R17 to R31, R18 to R32, R19 to R33, R20 to R34, R21 to R35, R22 to R36, R23 to R37, R24 to R38, R25 to R39, R26 to R40, R27 to R41, R28 to R42, R29 to R43, R30 to R44, R31 to R45, R5 to R46, RV1 to RV3, RV2 to RV4, U1 to U3, U3 to U4, U2 to U5
Connections:
- net VCO-TO-VCF renamed 5V?
- no-connect marks 8 -> 4

Commit message: ERC pass
Connections:
- net CV_BUS renamed CV
Changed lines of the file:
@@
 Connection ~ 7600 6450
 Text GLabel 5150 6850 0    50   Input ~ 0
-CV_BUS
+CV
 $Comp
 L Device:R R24

Commit message: Create pcb and other updates
Parts:
- removed unit 2 of U3
- C10, C8, C9: footprint (none) -> Capacitor_THT:CP_Radial_D6.3mm_P2.50mm
- C11, C6, C7: footprint (none) -> Capacitor_THT:C_Disc_D5.0mm_W2.5mm_P5.00mm
- D1, D2: footprint (none) -> Diode_THT:D_DO-15_P12.70mm_Horizontal
- K1: renamed from K4; footprint (none) -> Connector_PinSocket_2.54mm:PinSocket_1x03_P2.54mm_Vertical
- K2: renamed from K3; footprint (none) -> Connector_PinSocket_2.54mm:PinSocket_1x03_P2.54mm_Vertical
- K3: renamed from K2; footprint (none) -> Connector_PinSocket_2.54mm:PinSocket_1x03_P2.54mm_Vertical
- P2, P3, P4: footprint (none) -> Connector_PinSocket_2.54mm:PinSocket_1x03_P2.54mm_Vertical
- Q3, Q4, Q6, Q8: footprint (none) -> Package_TO_SOT_THT:TO-92L_Inline_Wide
- Q5, Q7: footprint Package_TO_SOT_THT:TO-92_Inline -> Package_TO_SOT_THT:TO-92L_Inline_Wide
- R18, R19, R20, R21, R23, R24, R25, R26, R27, R28, R29, R30, R31, R32, R33, R34, R35, R36, R37, R38, R39, R40, R41, R42, R43, R44, R45: footprint (none) -> Resistor_THT:R_Axial_DIN0207_L6.3mm_D2.5mm_P10.16mm_Horizontal
- RV16: renamed from R16; footprint (none) -> Potentiometer_THT:Potentiometer_Bourns_3296W_Vertical
- RV17: renamed from R17; footprint (none) -> Potentiometer_THT:Potentiometer_Bourns_3296W_Vertical
- RV22: renamed from R22; footprint (none) -> Potentiometer_THT:Potentiometer_Bourns_3296W_Vertical
- RV3, RV4: footprint (none) -> Potentiometer_THT:Potentiometer_Bourns_3296W_Vertical
- RV46: renamed from R46; footprint (none) -> Potentiometer_THT:Potentiometer_Bourns_3296W_Vertical
- U3: footprint (none) -> Package_DIP:DIP-14_W7.62mm_Socket_LongPads; symbol 74xx_IEEE:7413 -> janel-panel:7413
- U4: footprint (none) -> Package_DIP:DIP-14_W7.62mm_Socket_LongPads
- U5: footprint (none) -> Package_DIP:DIP-14_W7.62mm_Socket_LongPads; symbol 74xx_IEEE:7490 -> janel-panel:7490
Connections:
- net 5V? is gone; now on net LFO_OUT: P4.3, R30.1
- net VCC is gone; now on net +5V: U5.5 (VCC)
- net VDD is gone; now on net +5V: U3.14 (VDD)
- net VSS is gone; now on net GND: U3.7 (VSS)
- net +5V: now also R19.2; no longer R19.1
- net LFO_OUT: no longer R40.1, R41.1, R42.1
- net at R27.1: now also U3.8
- net at D1.2 (A), D2.2 (A), R31.1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: now also U3.9
- new net: R19.1, U3.10, U3.12, U3.13
- new net NOISE_LEVEL: R40.1, R41.1, R42.1
Other:
- moved on the sheet: C6, D1, D2, R19, R44, RV16
