File: LFO.kicad_sch (KiCad schematic)
At the start: 15 parts, among them K4 SW_SPDT, P1 100k, U5 uA741-DIP14, U6 UA747

Commit message: Fix PCB errors
Parts:
- added C_Sin1 (x6): Conn_01x01, Connector_PinHeader_2.54mm:PinHeader_1x01_P2.54mm_Vertical, symbol Connector_Generic:Conn_01x01
Connections:
- net LFO_OUT: now also C_Sin1.1 (Pin_1)
- net at P1.1, R9.1, U6.12: now also C_Sin1.1 (Pin_1)
- net at P1.3, R14.2: now also C_Sin1.1 (Pin_1)
- net at P1.2, R12.2: now also C_Sin1.1 (Pin_1)
- net at K4.1 (A), R7.2: now also C_Sin1.1 (Pin_1)
- net at K4.3 (C), R10.2: now also C_Sin1.1 (Pin_1)
Other:
- moved on the sheet: U6A
