File: VCO.kicad_sch (KiCad schematic)
At the start: 56 parts, among them K1 SW_SPST, K2 SW_SPST, K3 SW_SPST, P2 100k, P3 100k, P4 4k7, Q3 BC184, Q4 BC183B, Q5 BF244B, Q6 BC184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

Commit message: Fix PCB errors
Parts:
- added C_Sin1 (x12): Conn_01x01, Connector_PinHeader_2.54mm:PinHeader_1x01_P2.54mm_Vertical, symbol Connector_Generic:Conn_01x01
- C9: footprint Capacitor_THT:CP_Radial_D6.3mm_P2.50mm -> Capacitor_THT:CP_Radial_D8.0mm_P5.00mm
Connections:
- net LFO_OUT: now also C_Sin1.1 (Pin_1)
- net at RV22.3, RV3.3: now also C_Sin1.1 (Pin_1)
- net at C8.2, K3.1 (A): now also C_Sin1.1 (Pin_1)
- net at K3.2 (B), R40.2: now also C_Sin1.1 (Pin_1)
- net at C9.2, K2.1 (A): now also C_Sin1.1 (Pin_1)
- net at K2.2 (B), R41.2: now also C_Sin1.1 (Pin_1)
- net at C10.2, K1.1 (A): now also C_Sin1.1 (Pin_1)
- net at K1.2 (B), R42.2: now also C_Sin1.1 (Pin_1)
- net at Q3.3 (E), Q5.2 (G), Q8.2 (C)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: now also RV4.1; no longer RV4.3
- net at C6.1: now also RV4.3; no longer RV4.1
- net at P2.2, R20.2: now also C_Sin1.1 (Pin_1)
- net at P3.3, R25.2, R28.1: now also C_Sin1.1 (Pin_1)
- net at P3.2, R23.1: now also C_Sin1.1 (Pin_1)
- net at P4.2, R38.2: now also C_Sin1.1 (Pin_1)
Other:
- moved on the sheet: K1, K2, K3, P2, P4, R40, R41, R42, RV17, RV4
